File: hardware/logicboard/p1-001.brd (EAGLE design)
At the start: 47 x 72 mm, 24 parts, among them IC1 74LS07N

Commit message: Reserve pins.
Parts:
- moved RSV 61.9 mm to (29.2, 68.6), turned to 0 degrees
Routing:
- net LD9: track 180.8 -> 95.3 mm, vias 2 -> 3
- net LD11: track 69.5 -> 154.7 mm, vias 3 -> 2
- net D12: track 19.4 -> 84.7 mm, vias 0 -> 3
- net LD8: track 59.8 -> 119.7 mm, vias 0 -> 2
- net D11: track 19.9 -> 78.0 mm, vias 0 -> 1
- net LD5: track 31.3 -> 83.1 mm, vias 0 -> 3
- net D6: track 28.6 -> 71.1 mm, vias 0 -> 1
- net VDD: track 106.1 -> 72.0 mm
- net LD10: track 83.8 -> 53.9 mm, vias 5 -> 3
- net LD12: track 55.7 -> 82.3 mm
- net D5: track 26.6 -> 51.6 mm, vias 1 -> 3
- net SDA: track 102.8 -> 123.9 mm
- net D4: track 29.4 -> 48.1 mm, vias 1 -> 0
- net N$5: track 88.2 -> 70.0 mm, vias 7 -> 1
- net RX: track 78.9 -> 61.1 mm, vias 2 -> 3
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- removed copper zone on layer 1, net GND
- removed copper zone on layer 16, net GND

Commit message: Reserve pins.
Parts:
- RSV: device SparkFun-Connectors:1X05_1.27MM -> pinhead:1X05
- moved RSV 5.08 mm to (34.3, 68.6)
Routing:
- net LD11: track 154.7 -> 79.3 mm
- net SDA: track 123.9 -> 72.0 mm, vias 3 -> 1
- net LD8: track 119.7 -> 68.6 mm, vias 2 -> 0
- net VCC: track 195.7 -> 232.4 mm
- net LD9: track 95.3 -> 61.8 mm, vias 3 -> 2
- net D4: track 48.1 -> 79.4 mm, vias 0 -> 1
- net VDD: track 72.0 -> 91.9 mm, vias 2 -> 1
- net LD5: track 83.1 -> 63.3 mm, vias 3 -> 6
- net D11: track 78.0 -> 92.7 mm, vias 1 -> 2
- net N$3: track 94.6 -> 80.2 mm
- net LD6: track 61.9 -> 48.5 mm, vias 1 -> 0
- net V3V: track 39.4 -> 47.9 mm, vias 1 -> 0
- net GND: track 204.3 -> 195.9 mm, vias 3 -> 1
- net LD12: track 82.3 -> 74.2 mm, vias 4 -> 6
- net D12: track 84.7 -> 90.7 mm, vias 3 -> 1
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- added copper zone on layer 1, net GND
- added copper zone on layer 16, net GND
