File: hardware/logicboard/p1dc-001.sch (EAGLE design)
At the start: 40 parts, among them IC2 74LS595N, J0 DC24V, Q1 60V/32A/35mΩ, Q2 60V/32A/35mΩ, Q3 60V/32A/35mΩ, Q4 60V/32A/35mΩ, Q5 60V/32A/35mΩ, Q6 60V/32A/35mΩ, Q7 60V/32A/35mΩ, Q8 60V/32A/35mΩ

Commit message: Working.
Connections:
- net D1 renamed Q1
- net D2 renamed Q2
- net D3 renamed Q3
- net D4 renamed Q4
- net D6 renamed Q6
- net D7 renamed Q7
- net D8 renamed Q8
- new net Q5: IC2A.QE
- net D5: no longer IC2A.QE
Changed lines of the file:
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@@
 </segment>
 </net>
-<net name="D1" class="0">
+<net name="Q1" class="0">
 <segment>
 <wire x1="5.08" y1="149.86" x2="2.54" y2="149.86" width="0.1524" layer="91"/>
@@
 </segment>
 </net>
-<net name="D2" class="0">
+<net name="Q2" class="0">
 <segment>
 <wire x1="5.08" y1="111.76" x2="2.54" y2="111.76" width="0.1524" layer="91"/>
@@
 </segment>
 </net>
-<net name="D3" class="0">
+<net name="Q3" class="0">
 <segment>
 <wire x1="5.08" y1="73.66" x2="2.54" y2="73.66" width="0.1524" layer="91"/>
@@
 </segment>
 </net>
-<net name="D4" class="0">
+<net name="Q4" class="0">
 <segment>
 <wire x1="5.08" y1="35.56" x2="2.54" y2="35.56" width="0.1524" layer="91"/>
@@
 <pinref part="RN1" gate="E" pin="1"/>
 </segment>
-<segment>
-<pinref part="IC2" gate="A" pin="QE"/>
-<wire x1="213.36" y1="76.2" x2="215.9" y2="76.2" width="0.1524" layer="91"/>
-<label x="215.9" y="76.2" size="0.8128" layer="95" xref="yes"/>
-</segment>
-</net>
-<net name="D6" class="0">
+</net>
+<net name="Q6" class="0">
 <segment>
 <wire x1="88.9" y1="111.76" x2="86.36" y2="111.76" width="0.1524" layer="91"/>
@@
 </segment>
 </net>
-<net name="D7" class="0">
+<net name="Q7" class="0">
 <segment>
 <wire x1="88.9" y1="73.66" x2="86.36" y2="73.66" width="0.1524" layer="91"/>
@@
 <wire x1="213.36" y1="71.12" x2="215.9" y2="71.12" width="0.1524" layer="91"/>
 <label x="215.9" y="71.12" size="0.8128" layer="95" xref="yes"/>
-</segment>
-</net>
-<net name="D8" class="0">
-<segment>
-<wire x1="88.9" y1="35.56" x2="86.36" y2="35.56" width="0.1524" layer="91"/>
-<label x="86.36" y="35.56" size="0.8128" layer="95" rot="R180" xref="yes"/>
-<pinref part="RN1" gate="H" pin="1"/>
-</segment>
-<segment>
-<pinref part="IC2" gate="A" pin="QH"/>
-<wire x1="213.36" y1="68.58" x2="215.9" y2="68.58" width="0.1524" layer="91"/>
-<label x="215.9" y="68.58" size="0.8128" layer="95" xref="yes"/>
 </segment>
 </net>
@@
 </segment>
 </net>
+<net name="Q5" class="0">
+<segment>
+<pinref part="IC2" gate="A" pin="QE"/>
+<wire x1="213.36" y1="76.2" x2="215.9" y2="76.2" width="0.1524" layer="91"/>
+<label x="215.9" y="76.2" size="0.8128" layer="95" xref="yes"/>
+</segment>
+</net>
+<net name="Q8" class="0">
+<segment>
+<pinref part="IC2" gate="A" pin="QH"/>
+<wire x1="213.36" y1="68.58" x2="215.9" y2="68.58" width="0.1524" layer="91"/>
+<label x="215.9" y="68.58" size="0.8128" layer="95" xref="yes"/>
+</segment>
+<segment>
+<wire x1="88.9" y1="35.56" x2="86.36" y2="35.56" width="0.1524" layer="91"/>
+<label x="86.36" y="35.56" size="0.8128" layer="95" rot="R180" xref="yes"/>
+<pinref part="RN1" gate="H" pin="1"/>
+</segment>
+</net>
