File: hardware/logicboard/p1dc-001.brd (EAGLE design)
At the start: 95 x 72 mm, 40 parts, among them IC2 74LS595N, J0 DC24V, Q1 60V/32A/35mΩ, Q2 60V/32A/35mΩ, Q3 60V/32A/35mΩ, Q4 60V/32A/35mΩ, Q5 60V/32A/35mΩ, Q6 60V/32A/35mΩ, Q7 60V/32A/35mΩ, Q8 60V/32A/35mΩ

Commit message: Board design.
Parts:
- moved U$1 86.3 mm to (14.0, 66.0)
- moved LOGO1 7.81 mm to (84.0, 5.00)
- moved C3 4.00 mm to (15.0, 10.0)
- moved C4 4.00 mm to (11.0, 10.0)
- moved IC1 1.00 mm to (20.0, 2.00)
Routing:
- net D6: track 26.8 -> 49.7 mm
- net SCLK: track 142.9 -> 121.5 mm, vias 1 -> 4
- net GND: track 304.4 -> 284.2 mm, vias 0 -> 2
- net VCC/2: track 150.0 -> 163.1 mm, vias 2 -> 1
- net +24V: track 240.6 -> 249.3 mm, vias 3 -> 2
- net N$16: track 75.0 -> 81.0 mm
- net N$9: track 106.9 -> 112.1 mm
- net RCLK: track 117.5 -> 121.9 mm, vias 3 -> 0
- net N$6: track 128.9 -> 124.5 mm, vias 1 -> 2
- net N$15: track 45.0 -> 40.5 mm, vias 0 -> 1
- net SIN: track 37.4 -> 41.5 mm, vias 0 -> 1
- net VCC: track 125.6 -> 129.6 mm, vias 6 -> 2
- net N$21: track 35.9 -> 32.1 mm
- net IC2: track 119.0 -> 122.5 mm
- net GNDA: track 195.8 -> 199.1 mm, vias 2 -> 3
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- added copper zone on layer 1, net GND
- added copper zone on layer 16, net GND
Other:
- board text added: "Pineapple I dc 1.0.0-X"
- board text removed: "Cat-8 1.0.0-X"

Commit message: Working.
Connections:
- net D1 renamed Q1
- net D2 renamed Q2
- net D3 renamed Q3
- net D4 renamed Q4
- net D6 renamed Q6
- net D7 renamed Q7
- net D8 renamed Q8
- new net Q5: IC2.4
- net D5: no longer IC2.4
Changed lines of the file:
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@@
 <via x="16.6878" y="49.8348" extent="1-16" drill="0.3048"/>
 </signal>
-<signal name="D1">
+<signal name="Q1">
 <contactref element="RN1" pad="1"/>
 <contactref element="IC2" pad="15"/>
@@
 <wire x1="32.766" y1="55.3212" x2="32.81" y2="55.35" width="0.1524" layer="1"/>
 </signal>
-<signal name="D2">
+<signal name="Q2">
 <contactref element="RN1" pad="2"/>
 <contactref element="IC2" pad="1"/>
@@
 <wire x1="25.2222" y1="57.8358" x2="25.19" y2="57.89" width="0.1524" layer="16"/>
 </signal>
-<signal name="D3">
+<signal name="Q3">
 <contactref element="RN1" pad="3"/>
 <contactref element="IC2" pad="2"/>
@@
 <wire x1="25.2222" y1="55.3212" x2="25.19" y2="55.35" width="0.1524" layer="16"/>
 </signal>
-<signal name="D4">
+<signal name="Q4">
 <contactref element="RN1" pad="4"/>
 <contactref element="IC2" pad="3"/>
@@
 <signal name="D5">
 <contactref element="RN1" pad="5"/>
-<contactref element="IC2" pad="4"/>
 <wire x1="25.146" y1="25.3746" x2="25.146" y2="24.765" width="0.1524" layer="1"/>
 <wire x1="23.241" y1="27.2796" x2="25.146" y2="25.3746" width="0.1524" layer="1"/>
@@
 <wire x1="25.146" y1="50.2158" x2="25.146" y2="49.8348" width="0.1524" layer="1"/>
 <wire x1="25.146" y1="24.765" x2="25.19" y2="24.73" width="0.1524" layer="1"/>
-<wire x1="25.146" y1="50.2158" x2="25.19" y2="50.27" width="0.1524" layer="1"/>
-</signal>
-<signal name="D6">
+</signal>
+<signal name="Q6">
 <contactref element="RN1" pad="6"/>
 <contactref element="IC2" pad="5"/>
@@
 <via x="18.0594" y="43.7388" extent="1-16" drill="0.3048"/>
 </signal>
-<signal name="D7">
+<signal name="Q7">
 <contactref element="RN1" pad="7"/>
 <contactref element="IC2" pad="6"/>
@@
 <wire x1="25.2222" y1="19.6596" x2="25.19" y2="19.65" width="0.1524" layer="16"/>
 <wire x1="25.146" y1="45.1866" x2="25.19" y2="45.19" width="0.1524" layer="16"/>
-</signal>
-<signal name="D8">
-<contactref element="RN1" pad="8"/>
-<contactref element="IC2" pad="7"/>
-<wire x1="25.2222" y1="17.7546" x2="25.2222" y2="17.145" width="0.1524" layer="16"/>
-<wire x1="29.1846" y1="21.717" x2="25.2222" y2="17.7546" width="0.1524" layer="16"/>
-<wire x1="29.1846" y1="38.6334" x2="29.1846" y2="21.717" width="0.1524" layer="16"/>
-<wire x1="25.2222" y1="42.5958" x2="29.1846" y2="38.6334" width="0.1524" layer="16"/>
-<wire x1="25.2222" y1="17.145" x2="25.19" y2="17.11" width="0.1524" layer="16"/>
-<wire x1="25.2222" y1="42.5958" x2="25.19" y2="42.65" width="0.1524" layer="16"/>
 </signal>
 <signal name="N$1">
@@
 <wire x1="9.7536" y1="41.148" x2="9.73" y2="41.08" width="0.1524" layer="16"/>
 </signal>
+<signal name="Q5">
+<contactref element="IC2" pad="4"/>
+</signal>
+<signal name="Q8">
+<contactref element="IC2" pad="7"/>
+<contactref element="RN1" pad="8"/>
+<wire x1="25.2222" y1="17.7546" x2="25.2222" y2="17.145" width="0.1524" layer="16"/>
+<wire x1="29.1846" y1="21.717" x2="25.2222" y2="17.7546" width="0.1524" layer="16"/>
+<wire x1="29.1846" y1="38.6334" x2="29.1846" y2="21.717" width="0.1524" layer="16"/>
+<wire x1="25.2222" y1="42.5958" x2="29.1846" y2="38.6334" width="0.1524" layer="16"/>
+<wire x1="25.2222" y1="17.145" x2="25.19" y2="17.11" width="0.1524" layer="16"/>
+<wire x1="25.2222" y1="42.5958" x2="25.19" y2="42.65" width="0" layer="19" extent="16-16"/>
+</signal>
 </signals>

Commit message: Clean up of the board design of Pineapple I dc driver.
Parts:
- moved SV2 74.3 mm to (11.0, 50.0), turned to 90 degrees
- moved U$1 70.5 mm to (47.5, 4.00)
- moved DZ1 49.8 mm to (88.0, 36.0), turned to 270 degrees
- moved LOGO1 36.8 mm to (47.5, 10.0)
- moved SV1 14.0 mm to (11.0, 22.0)
- moved C1 8.25 mm to (37.0, 8.00)
- moved C2 8.25 mm to (33.0, 8.00)
- moved IC1 6.40 mm to (25.0, 6.00)
- moved C3 2.83 mm to (17.0, 8.00)
- moved C4 2.83 mm to (13.0, 8.00)
Routing:
- net IC2: track 122.5 -> 28.8 mm
- net IC1: track 119.7 -> 28.8 mm
- net RCLK: track 121.9 -> 62.3 mm
- net SCLK: track 121.5 -> 63.8 mm, vias 4 -> 1
- net N$7: track 36.0 -> 88.0 mm, vias 0 -> 1
- net VCC: track 129.6 -> 79.8 mm, vias 2 -> 1
- net N$10: track 28.7 -> 77.4 mm
- net N$4: track 45.0 -> 88.7 mm, vias 0 -> 1
- net SOUT: track 64.2 -> 26.3 mm, vias 2 -> 0
- net VCC/2: track 163.1 -> 131.8 mm, vias 1 -> 0
- net D5: track 29.1 -> 0.00 mm
- net +24V: track 249.3 -> 224.1 mm
- net GNDA: track 199.1 -> 174.3 mm, vias 3 -> 1
- net N$9: track 112.1 -> 87.8 mm
- net N$12: track 103.5 -> 83.4 mm
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- removed copper zone on layer 1, net GND
- removed copper zone on layer 16, net GND
