File: hardware/logicboard/p1ac-001.sch (EAGLE design)
At the start: 30 parts, among them IC1 74LS595N, IC2 74LS595N, K1 AQG12105, K10 AQG12105, K11 AQG12105, K12 AQG12105, K13 AQG12105, K14 AQG12105, K15 AQG12105, K16 AQG12105, K2 AQG12105, K3 AQG12105, K4 AQG12105, K5 AQG12105, K6 AQG12105, K7 AQG12105, K8 AQG12105, K9 AQG12105

Commit message: First shot.
Parts:
- removed IC2: 74LS595N, 74xx-us:74LS595N
- removed K10, K11, K12, K13, K14, K15, K16, K9: AQG12105, relay:AQG12105
- removed SV1: (no value), con-ml:ML34L
- removed ULN2: (no value), SparkFun-IC-Special-Function:ULN2803DIP
- added DZ1: LB10, led:LB10
- added J2, J3, J4, J5, J6, J7, J8, J9: (no value), SparkFun-Connectors:CONN_02POLAR
- added RN1: (no value), resistor-dil:8R-N
- J1: device Seeed-Connector:JACK-DC-005'DC-005' -> SparkFun-Connectors:CONN_02POLAR
Connections:
- net S1 renamed Q1
- net S2 renamed Q2
- net S3 renamed Q3
- net S4 renamed Q4
- net S6 renamed Q6
- net S7 renamed Q7
- net S8 renamed Q8
- removed net +24V: J1.+, K1.DS1, K10.DS1, K11.DS1, K12.DS1, K13.DS1, K14.DS1, K15.DS1, K16.DS1, K2.DS1, K3.DS1, K4.DS1, K5.DS1, K6.DS1, K7.DS1, K8.DS1, K9.DS1
- removed net N$9: IC1A.QH*, IC2A.SER
- removed net R10: K10.K, ULN2.17
- removed net R11: K11.K, ULN2.16
- removed net R12: K12.K, ULN2.15
- removed net R13: K13.K, ULN2.14
- removed net R14: K14.K, ULN2.13
- removed net R15: K15.K, ULN2.12
- removed net R16: K16.K, ULN2.11
- removed net R9: K9.K, ULN2.18
- removed net S10: IC2A.QB, ULN2.2
- removed net S11: IC2A.QC, ULN2.3
- removed net S12: IC2A.QD, ULN2.4
- removed net S13: IC2A.QE, ULN2.5
- removed net S14: IC2A.QF, ULN2.6
- removed net S15: IC2A.QG, ULN2.7
- removed net S16: IC2A.QH, ULN2.8
- removed net S9: IC2A.QA, ULN2.1
- removed net X10: K10.DS2, SV1.19
- removed net X11: K11.DS2, SV1.21
- removed net X12: K12.DS2, SV1.23
- removed net X13: K13.DS2, SV1.25
- removed net X14: K14.DS2, SV1.27
- removed net X15: K15.DS2, SV1.29
- removed net X16: K16.DS2, SV1.31
- removed net X9: K9.DS2, SV1.17
- new net AC1: J9.1, K1.DS1, K2.DS1, K3.DS1, K4.DS1, K5.DS1, K6.DS1, K7.DS1, K8.DS1
- new net AC2: J1.2, J2.2, J3.2, J4.2, J5.2, J6.2, J7.2, J8.2, J9.2
- new net N$1: IC1A.QH*
- new net N$2: DZ1-1.A, RN1A.2
- new net Q5: ULN1.5
- net CLR: no longer IC2A.SCL
- net GND: no longer IC2A.G, J1.-, J1.CDN, SV1.10, SV1.12, SV1.14, SV1.16, SV1.18, SV1.2, SV1.20, SV1.22, SV1.24, SV1.26, SV1.28, SV1.30, SV1.32, SV1.33, SV1.34, SV1.4, SV1.6, SV1.8, ULN2.9
- net R1: now also DZ1-1.C
- net RCLK: no longer IC2A.RCK
- net S5: no longer ULN1.5
- net SCLK: no longer IC2A.SCK
- net SOUT: no longer IC2A.QH*
- net VCC: now also RN1A.1; no longer K10.A, K11.A, K12.A, K13.A, K14.A, K15.A, K16.A, K9.A, ULN2.10
- net X1: now also J1.1; no longer SV1.1
- net X2: now also J2.1; no longer SV1.3
- net X3: now also J3.1; no longer SV1.5
- net X4: now also J4.1; no longer SV1.7
- net X5: now also J5.1; no longer SV1.9
- net X6: now also J6.1; no longer SV1.11
- net X7: now also J7.1; no longer SV1.13
- net X8: now also J8.1; no longer SV1.15
Other:
- moved on the sheet: ULN1

Commit message: Working.
Connections:
- removed net N$1: IC1A.QH*
- removed net S5: IC1A.QE
- new net N$10: DZ1-4.A, RN1D.2
- new net N$13: DZ1-5.A, RN1E.2
- new net N$16: DZ1-6.A, RN1F.2
- new net N$19: DZ1-7.A, RN1G.2
- new net N$22: DZ1-8.A, RN1H.2
- new net N$4: DZ1-2.A, RN1B.2
- new net N$7: DZ1-3.A, RN1C.2
- net Q5: now also IC1A.QE
- net R2: now also DZ1-2.C
- net R3: now also DZ1-3.C
- net R4: now also DZ1-4.C
- net R5: now also DZ1-5.C
- net R6: now also DZ1-6.C
- net R7: now also DZ1-7.C
- net R8: now also DZ1-8.C
- net SOUT: now also IC1A.QH*
- net VCC: now also RN1B.1, RN1C.1, RN1D.1, RN1E.1, RN1F.1, RN1G.1, RN1H.1
Other:
- moved on the sheet: DZ1-10, DZ1-2, DZ1-3, DZ1-4, DZ1-5, DZ1-6, DZ1-7, DZ1-8, DZ1-9, J1, J2, J3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

Commit message: Board design of Pineapple I ac driver.
Parts:
- removed C4: (no value), resistor:C-EU025-024X044
Connections:
- net GND: no longer C4.2
- net VCC: no longer C4.1
Other:
- moved on the sheet: J5, J6
Changed lines of the file:
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@@
 <part name="C2" library="resistor" library_urn="urn:adsk.eagle:library:348" deviceset="C-EU" device="025-024X044" package3d_urn="urn:adsk.eagle:package:26149/1"/>
 <part name="C3" library="resistor" library_urn="urn:adsk.eagle:library:348" deviceset="C-EU" device="025-024X044" package3d_urn="urn:adsk.eagle:package:26149/1"/>
-<part name="C4" library="resistor" library_urn="urn:adsk.eagle:library:348" deviceset="C-EU" device="025-024X044" package3d_urn="urn:adsk.eagle:package:26149/1"/>
 <part name="SUPPLY1" library="supply2" deviceset="GND" device=""/>
 <part name="P+1" library="supply1" library_urn="urn:adsk.eagle:library:371" deviceset="VCC" device=""/>
@@
 <attribute name="VALUE" x="21.844" y="25.781" size="1.778" layer="96"/>
 </instance>
-<instance part="C4" gate="G$1" x="27.94" y="30.48" smashed="yes">
-<attribute name="NAME" x="29.464" y="30.861" size="1.778" layer="95"/>
-<attribute name="VALUE" x="29.464" y="25.781" size="1.778" layer="96"/>
-</instance>
 <instance part="SUPPLY1" gate="GND" x="5.08" y="17.78" smashed="yes"/>
 <instance part="P+1" gate="VCC" x="7.62" y="78.74" smashed="yes">
@@
 <attribute name="NAME" x="215.9" y="96.012" size="1.778" layer="95" font="vector" rot="R180"/>
 </instance>
-<instance part="J5" gate="G$1" x="215.9" y="83.82" smashed="yes" rot="R180">
-<attribute name="VALUE" x="218.44" y="88.646" size="1.778" layer="96" font="vector" rot="R180"/>
-<attribute name="NAME" x="218.44" y="78.232" size="1.778" layer="95" font="vector" rot="R180"/>
-</instance>
-<instance part="J6" gate="G$1" x="210.82" y="66.04" smashed="yes" rot="R180">
-<attribute name="VALUE" x="213.36" y="70.866" size="1.778" layer="96" font="vector" rot="R180"/>
-<attribute name="NAME" x="213.36" y="60.452" size="1.778" layer="95" font="vector" rot="R180"/>
+<instance part="J5" gate="G$1" x="213.36" y="83.82" smashed="yes" rot="R180">
+<attribute name="VALUE" x="215.9" y="88.646" size="1.778" layer="96" font="vector" rot="R180"/>
+<attribute name="NAME" x="215.9" y="78.232" size="1.778" layer="95" font="vector" rot="R180"/>
+</instance>
+<instance part="J6" gate="G$1" x="213.36" y="66.04" smashed="yes" rot="R180">
+<attribute name="VALUE" x="215.9" y="70.866" size="1.778" layer="96" font="vector" rot="R180"/>
+<attribute name="NAME" x="215.9" y="60.452" size="1.778" layer="95" font="vector" rot="R180"/>
 </instance>
 <instance part="J7" gate="G$1" x="213.36" y="48.26" smashed="yes" rot="R180">
@@
 <wire x1="5.08" y1="25.4" x2="5.08" y2="22.86" width="0.1524" layer="91"/>
 <wire x1="5.08" y1="22.86" x2="12.7" y2="22.86" width="0.1524" layer="91"/>
-<pinref part="C4" gate="G$1" pin="2"/>
 <wire x1="12.7" y1="22.86" x2="20.32" y2="22.86" width="0.1524" layer="91"/>
-<wire x1="20.32" y1="22.86" x2="27.94" y2="22.86" width="0.1524" layer="91"/>
-<wire x1="27.94" y1="22.86" x2="27.94" y2="25.4" width="0.1524" layer="91"/>
 <pinref part="C2" gate="G$1" pin="2"/>
 <wire x1="12.7" y1="25.4" x2="12.7" y2="22.86" width="0.1524" layer="91"/>
@@
 <pinref part="C3" gate="G$1" pin="2"/>
 <wire x1="20.32" y1="25.4" x2="20.32" y2="22.86" width="0.1524" layer="91"/>
-<junction x="20.32" y="22.86"/>
 <wire x1="5.08" y1="22.86" x2="5.08" y2="20.32" width="0.1524" layer="91"/>
 <junction x="5.08" y="22.86"/>
@@
 </segment>
 </net>
-<net name="X1" class="0">
+<net name="X1" class="2">
 <segment>
 <pinref part="K1" gate="A" pin="DS2"/>
@@
 </segment>
 </net>
-<net name="X2" class="0">
+<net name="X2" class="2">
 <segment>
 <pinref part="K2" gate="A" pin="DS2"/>
@@
 </segment>
 </net>
-<net name="X3" class="0">
+<net name="X3" class="2">
 <segment>
 <pinref part="K3" gate="A" pin="DS2"/>
@@
 </segment>
 </net>
-<net name="X4" class="0">
+<net name="X4" class="2">
 <segment>
 <pinref part="K4" gate="A" pin="DS2"/>
@@
 </segment>
 </net>
-<net name="X5" class="0">
+<net name="X5" class="2">
 <segment>
 <pinref part="K5" gate="A" pin="DS2"/>
-<wire x1="200.66" y1="83.82" x2="208.28" y2="83.82" width="0.1524" layer="91"/>
+<wire x1="200.66" y1="83.82" x2="205.74" y2="83.82" width="0.1524" layer="91"/>
 <pinref part="J5" gate="G$1" pin="1"/>
 </segment>
 </net>
-<net name="X6" class="0">
+<net name="X6" class="2">
 <segment>
 <pinref part="K6" gate="A" pin="DS2"/>
-<wire x1="200.66" y1="66.04" x2="203.2" y2="66.04" width="0.1524" layer="91"/>
+<wire x1="200.66" y1="66.04" x2="205.74" y2="66.04" width="0.1524" layer="91"/>
 <pinref part="J6" gate="G$1" pin="1"/>
 </segment>
 </net>
-<net name="X7" class="0">
+<net name="X7" class="2">
 <segment>
 <pinref part="K7" gate="A" pin="DS2"/>
@@
 </segment>
 </net>
-<net name="X8" class="0">
+<net name="X8" class="2">
 <segment>
 <pinref part="K8" gate="A" pin="DS2"/>
@@
 <wire x1="5.08" y1="33.02" x2="5.08" y2="35.56" width="0.1524" layer="91"/>
 <wire x1="5.08" y1="35.56" x2="12.7" y2="35.56" width="0.1524" layer="91"/>
-<pinref part="C4" gate="G$1" pin="1"/>
 <wire x1="12.7" y1="35.56" x2="20.32" y2="35.56" width="0.1524" layer="91"/>
-<wire x1="20.32" y1="35.56" x2="27.94" y2="35.56" width="0.1524" layer="91"/>
-<wire x1="27.94" y1="35.56" x2="27.94" y2="33.02" width="0.1524" layer="91"/>
 <pinref part="C3" gate="G$1" pin="1"/>
 <wire x1="20.32" y1="33.02" x2="20.32" y2="35.56" width="0.1524" layer="91"/>
-<junction x="20.32" y="35.56"/>
 <pinref part="C2" gate="G$1" pin="1"/>
 <wire x1="12.7" y1="33.02" x2="12.7" y2="35.56" width="0.1524" layer="91"/>
@@
 </segment>
 </net>
-<net name="AC2" class="0">
+<net name="AC2" class="2">
 <segment>
 <pinref part="J1" gate="G$1" pin="2"/>
@@
 <segment>
 <pinref part="J5" gate="G$1" pin="2"/>
-<wire x1="208.28" y1="81.28" x2="203.2" y2="81.28" width="0.1524" layer="91"/>
+<wire x1="205.74" y1="81.28" x2="203.2" y2="81.28" width="0.1524" layer="91"/>
 <label x="203.2" y="81.28" size="0.8128" layer="95" rot="R180" xref="yes"/>
 </segment>
 <segment>
 <pinref part="J6" gate="G$1" pin="2"/>
-<wire x1="203.2" y1="63.5" x2="200.66" y2="63.5" width="0.1524" layer="91"/>
-<label x="200.66" y="63.5" size="0.8128" layer="95" rot="R180" xref="yes"/>
-</segment>
-<segment>
+<wire x1="205.74" y1="63.5" x2="203.2" y2="63.5" width="0.1524" layer="91"/>
+<label x="203.2" y="63.5" size="0.8128" layer="95" rot="R180" xref="yes"/>
+</segment>
+<segment>
